Commit message: Fix the naming problems.

File: robots/Crawler_URDF_V2.URDF (robot description, URDF)
Before this commit: robot IWAMP_URDF_151021.SLDASM, 10 links, 9 joints
Links:
- link arm_pitch_link: geometry collision mesh filename=package://Crawler_URDF_V2/meshes/arm_pitch_link.STL; visual mesh filename=package://Crawler_URDF_V2/meshes/arm_pitch_link.STL
- link arm_prismatic_link: geometry collision mesh filename=package://Crawler_URDF_V2/meshes/arm_prismatic_link.STL; visual mesh filename=package://Crawler_URDF_V2/meshes/arm_prismatic_link.STL
- link arm_yaw_link: geometry collision mesh filename=package://Crawler_URDF_V2/meshes/arm_yaw_link.STL; visual mesh filename=package://Crawler_URDF_V2/meshes/arm_yaw_link.STL
- link chasis_link: geometry collision mesh filename=package://Crawler_URDF_V2/meshes/chasis_link.STL; visual mesh filename=package://Crawler_URDF_V2/meshes/chasis_link.STL
- link cmass_left_link: geometry collision mesh filename=package://Crawler_URDF_V2/meshes/cmass_left_link.STL; visual mesh filename=package://Crawler_URDF_V2/meshes/cmass_left_link.STL
- link cmass_right_link: geometry collision mesh filename=package://Crawler_URDF_V2/meshes/cmass_right_link.STL; visual mesh filename=package://Crawler_URDF_V2/meshes/cmass_right_link.STL
- link tool_link: geometry collision mesh filename=package://Crawler_URDF_V2/meshes/tool_link.STL; visual mesh filename=package://Crawler_URDF_V2/meshes/tool_link.STL
- link trans_base_link: geometry collision mesh filename=package://Crawler_URDF_V2/meshes/trans_base_link.STL; visual mesh filename=package://Crawler_URDF_V2/meshes/trans_base_link.STL
- link wrist_pitch_link: geometry collision mesh filename=package://Crawler_URDF_V2/meshes/wrist_pitch_link.STL; visual mesh filename=package://Crawler_URDF_V2/meshes/wrist_pitch_link.STL
- link wrist_row_link: geometry collision mesh filename=package://Crawler_URDF_V2/meshes/wrist_row_link.STL; visual mesh filename=package://Crawler_URDF_V2/meshes/wrist_row_link.STL

Commit message: Fix color bugs, and add V-REP files.

File: robots/Crawler_URDF_V2.URDF (robot description, URDF)
Before this commit: robot Crawler_URDF_V2, 10 links, 9 joints
Links:
- removed link wrist_row_link
- added link wrist_roll_link, mass 0.99835; collision mesh filename=package://Crawler_URDF_V2/meshes/wrist_roll_link.STL; visual mesh filename=package://Crawler_URDF_V2/meshes/wrist_roll_link.STL
- link arm_pitch_link: mass 1.85488275899258 -> 1.8549
- link arm_prismatic_link: mass 0.110019786871871 -> 0.11002
- link arm_yaw_link: mass 0.361799671756217 -> 0.3618
- link chasis_link: mass 9.63949891888311 -> 9.6395
- link cmass_left_link: mass 0.544396872641284 -> 0.5444
- link cmass_right_link: mass 0.544396872641284 -> 0.5444
- link tool_link: mass 0.999157186107062 -> 0.99916
- link trans_base_link: mass 1.52634919066965 -> 1.5263
- link wrist_pitch_link: mass 0.00528345401160869 -> 0.0052835
Joints:
- removed joint wrist_row_joint
- added joint wrist_roll_joint: type revolute, parent wrist_pitch_link, child wrist_roll_link, origin xyz=0 0.0127 0 rpy=1.0472 1.5708 0, axis 0 0.86603 0.5, limit lower=-0.5236 upper=0.5236 effort=0 velocity=0
- joint tool_joint: origin xyz=0 0.13895 0.0020772 rpy=1.5708 5.0343E-13 6.3761E-13 -> xyz=0 0.071274 -0.1193 rpy=0.5236 2.5158E-13 -4.363E-13; parent wrist_row_link -> wrist_roll_link
